File: BlockBox v2.sch (EAGLE design)
At the start: 214 parts, among them J100 TE-770966, Q100 TK3R1E04PL, Q101 TK3R1E04PL, Q102 IPP052N06L3 G, Q103 IPP052N06L3 G, Q104 IPP052N06L3 G, Q105 IPP052N06L3 G, Q106 TK3R1E04PL, Q200 SUP90142E-GE3, Q201 SUP90142E-GE3, Q202 BUK9Y43-60E, Q203 DMP4065S, SW100 PWRSW, U100 BQ77915, U101 MAX1737, U102 LM74700-Q1, U103 LM74700-Q1, U104 LM74700-Q1, U200 LM5022, U201 LM3488, U202 LM25085, U203 TPS54308, U204 LD39150DT33, U300 TAS5548, U301 TAS5634, U302 NCS20071

Commit message: Audio path done, MCU project added
Parts:
- added A400: BM83, BW-Active:BM83
- added C329, C330, C331, C332, C335, C337: 0.1µF, rcl:C-EUC0603
- added C333, C334, C336: 10µF, rcl:C-EUC0805
- added C338, C339: 18pF, rcl:C-EUC0603
- added C340, C342: 4.7nF, rcl:C-EUC0603
- added C341, C343: 47nF, rcl:C-EUC0603
- added R310: 1MΩ, resistor:R-US_R0603
- added R311, R312: 470Ω, resistor:R-US_R0603
- added R313: 10kΩ, resistor:R-US_R0603
- added U400: PIC32MZ-EF-100-I/PF, BW-Active:PIC32MZ-EF-100-I/PF
- added XDS1: NHD-3.5-320240FT-CON, BW-Active:NHD-3.5-320240FT-CON
- added Y300: 12.288MHz, BW-PassiveMechanical:HC49US-CRYSTAL
- L300, L301, L302, L303: device BW-PassiveMechanical:15153C -> BW-PassiveMechanical:1D14A
- R110, R113, R114, R115, R116, R118, R119, R120, R121, R126, R128, R200, R214, R218, R220, R301: device resistor:R-US_R0805 -> resistor:R-US_R0603
Connections:
- net N$1 renamed AMP_M2
- new net DSP_!MUTE: U300.!MUTE
- new net DSP_!PDN: U300.!PDN
- new net DSP_!RESET: U300.!RESET
- new net DSP_ASEL_EMO2: R313.2, U300.ASEL_EMO2
- new net DSP_EMO1: U300.EMO1
- new net DSP_PLL_FLTM: C342.1, C343.1, U300.PLL_FLTM
- new net DSP_PLL_FLTP: C340.2, R311.2, U300.PLL_FLTP
- new net DSP_PLL_FLTP_INT: C341.2, R311.1
- new net DSP_PLL_FPLM_INT: C343.2, R312.1
- new net DSP_SCL: U300.SCL
- new net DSP_SDA: U300.SDA
- new net DSP_VR_ANA: C340.1, C341.1, U300.VR_ANA
- new net DSP_VR_DIG: C335.1, C336.1, U300.VR_DIG
- new net DSP_VR_PWM: C337.1, U300.VR_PWM
- new net DSP_XTALI: C338.2, R310.2, U300.XTALI, Y300.2
- new net DSP_XTALO: C339.2, R310.1, U300.XTALO, Y300.1
- new net I2S_LRCLK: U300.LRCLK
- new net I2S_SCLK: U300.SCLK
- new net I2S_SD: U300.SDIN1
- net 3.3V: now also C329.1, C330.1, C331.1, C332.1, C333.1, C334.1, U300.!HP_SEL, U300.VDD
- net AMP_INPUT_A: now also U300.PWM_P_8; no longer U300.PWM_P_2
- net AMP_INPUT_B: now also U300.PWM_M_8; no longer U300.PWM_M_2
- net AMP_INPUT_C: now also U300.PWM_P_7; no longer U300.PWM_P_1
- net AMP_INPUT_D: now also U300.PWM_M_7; no longer U300.PWM_M_1
- net GND: now also C329.2, C330.2, C331.2, C332.2, C333.2, C334.2, C335.2, C336.2, C337.2, C338.1, C339.1, C342.2, R312.2, R313.1, U300.VSS

Commit message: MCU config done (for now), schematic base done
Parts:
- removed XDS1: NHD-3.5-320240FT-CON, BW-Active:NHD-3.5-320240FT-CON
- added C400, C409, C410, C411, C412, C413, C414, C415, C416, C417, C418, C419, C420: 0.1µF, rcl:C-EUC0603
- added C401, C402, C403, C404, C405, C406, C407: 15pF, rcl:C-EUC0603
- added C408: 0.1µF, rcl:C-EUC0805
- added C421, C422: 18pF, rcl:C-EUC0603
- added J400: ICSP, BW-Connectors:5P-1.27-POGO
- added J401: LED, BW-Connectors:GEN-4PIN
- added J402: SWLED, BW-Connectors:GEN-3PIN
- added J403: USB1, BW-Connectors:GEN-2PIN
- added J404: USB2, BW-Connectors:GEN-2PIN
- added J405, J406, J407: ZX62D-B-5PA8, BW-Connectors:ZX62D-B-5PA8
- added Q400, Q401, Q402, Q403: DMG2302UK, BW-Active:SOT23-N-MOSFET
- added Q404, Q405, Q406: NMOS, BW-Active:SOT23-N-MOSFET
- added R400, R402, R403, R404: 10kΩ, resistor:R-US_R0603
- added R401, R406: 1kΩ, resistor:R-US_R0603
- added R405: 1.69kΩ, resistor:R-US_R0603
- added RV400: 100kΩ, BW-PassiveMechanical:WIRED-POTENTIOMETER
- added SJ400: USB, jumper:SJ2W
- added SJ401: 3.3V-5V, jumper:SJ2W
- added SJ402: VBUS, jumper:SJ
- added SJ403: FTRESET, jumper:SJ
- added SJ404: USB-5V, jumper:SJ2W
- added SW400: VOL-, BW-PassiveMechanical:WIRED-SWITCH-NO
- added SW401: MFB, BW-PassiveMechanical:WIRED-SWITCH-NO
- added SW402: VOL+, BW-PassiveMechanical:WIRED-SWITCH-NO
- added SW403: BACK, BW-PassiveMechanical:WIRED-SWITCH-NO
- added SW404: PLAY, BW-PassiveMechanical:WIRED-SWITCH-NO
- added SW405: FWD, BW-PassiveMechanical:WIRED-SWITCH-NO
- added SW406: LCD_BL, BW-PassiveMechanical:WIRED-SWITCH-NO
- added SW407: LEDMODE, BW-PassiveMechanical:WIRED-SWITCH-U
- added SW408: SDA01H1S, BW-PassiveMechanical:SDA01H1S
- added U401: FT230XS, ftdichip:FT230XS
- added U402: NCS20071, BW-Active:NCS20071
- added U404: FSAL200MTC, BW-Active:FSAL200MTC
- added XDS400: NHD-3.5-320240FT-CON, BW-Active:NHD-3.5-320240FT-CON
- added Y400: 12MHz, BW-PassiveMechanical:HC49US-CRYSTAL
Connections:
- new net BM_!RST: A400.RST_N, U400.RD13
- new net BM_ADAP_IN: A400.ADAP_IN, SJ404.2
- new net BM_MFB: A400.MFB, U400.RF0
- new net BM_P3_4: A400.P3_4/UART_RTS, Q406.D
- new net BM_UART_RXD: A400.UART_RXD, U404A.A
- new net BM_UART_SWITCH: Q406.G, R402.2, SW408.1, U404M.S
- new net BM_UART_TXD: A400.UART_TXD, U404B.A
- new net BM_USB_D+: A400.DP, J406.D+
- new net BM_USB_D-: A400.DM, J406.D-
- new net BM_USB_VBUS: J406.VBUS, SJ404.1
- new net FT_!CTS: R403.2, U401.!CTS
- new net FT_!RESET: SJ403.2, U401.!RESET
- new net FT_RXD: U401.RXD, U404B.B2
- new net FT_TXD: U401.TXD, U404A.B2
- new net FT_USB_D+: J405.D+, U401.USBDP
- new net FT_USB_D-: J405.D-, U401.USBDM
- new net FT_USB_VBUS: J405.VBUS, SJ402.1
- new net FT_VBUS_SENSE: SJ402.2, U401.CBUS1
- new net LCD_!CS: U400.RC2, XDS400.!CS
- new net LCD_!INT: U400.RC4, XDS400.!INT
- new net LCD_!PD: U400.RC3, XDS400.!PD
- new net LCD_ADD_PIN: U400.RA5, XDS400.AUDIO_L
- new net LCD_BL_CTL: Q400.G, U400.RG15
- new net LCD_GND_BL: Q400.D, XDS400.GND_BL
- new net LCD_GPIO0: U400.RC1, XDS400.GPIO0/IO2
- new net LCD_GPIO1: U400.RE7, XDS400.GPIO1/IO3
- new net LCD_GPIO2: U400.RE6, XDS400.GPIO2
- new net LCD_GPIO3: U400.RE5, XDS400.GPIO3
- new net LCD_MISO: U400.RG7, XDS400.MISO/IO1
- new net LCD_MOSI: U400.RG8, XDS400.MOSI/IO0
- new net LCD_SCK: U400.RG6, XDS400.SCK
- new net LCD_VBL: SJ401.2, XDS400.VBL
- new net LED_B: J401D.P$1, Q403.D
- new net LED_G: J401B.P$1, Q401.D
- new net LED_R: J401C.P$1, Q402.D
- new net MCU_!MCLR: J400.1, R401.2, U400.!MCLR
- new net MCU_!MCLR!_FILT: C400.1, R400.1, R401.1
- new net MCU_BACK_SW: C404.2, SW403.1, U400.RG13
- new net MCU_BAT_SENSE: U400.RB6, U402.-IN, U402.OUT
- new net MCU_BAT_VDIV: R404.1, R405.2, U402.+IN
- new net MCU_FWD_SW: C402.2, SW405.1, U400.RE3
- new net MCU_LCD_BL_SW: C401.2, SW406.1, U400.RE4
- new net MCU_LED_B: Q403.G, U400.RB5
- new net MCU_LED_G: Q401.G, U400.RE8
- new net MCU_LED_MODE1: SW407.O, U400.RG9
- new net MCU_LED_MODE2: SW407.S, U400.RA0
- new net MCU_LED_POT: RV400.S, U400.RB4
- new net MCU_LED_R: Q402.G, U400.RE9
- new net MCU_MFB_SW: C406.2, SW401.1, U400.RG14
- new net MCU_OSC1: C421.2, U400.RC12, Y400.2
- new net MCU_OSC2: R406.2, U400.RC15
- new net MCU_OSC2_R: C422.2, R406.1, Y400.1
- new net MCU_PGC: J400.5, U400.RB1
- new net MCU_PGD: J400.4, U400.RB0
- new net MCU_PLAY_SW: C403.2, SW404.1, U400.RE2
- new net MCU_SWLED_MAIN: Q404.G, U400.RB3
- new net MCU_SWLED_PWR: Q405.G, U400.RB2
- new net MCU_UART_RX: U400.RD4, U404B.B1
- new net MCU_UART_TX: U400.RD5, U404A.B1
- new net MCU_USBID: J407.ID, U400.RF3
- new net MCU_USB_D+: J407.D+, U400.D+
- new net MCU_USB_D-: J407.D-, U400.D-
- new net MCU_USB_VBUS: J407.VBUS, U400.VBUS
- new net MCU_VOL+_SW: C405.2, SW402.1, U400.RG12
- new net MCU_VOL-_SW: C407.2, SW400.1, U400.RE1
- new net MCU_VUSB3V3: SJ400.2, U400.VUSB3V3
- new net SWLED_MAIN: J402B.P$1, Q404.D
- new net SWLED_PWR: J402C.P$1, Q405.D
- net 12V: now also J401A.P$1
- net 3.3V: now also A400.BAT_IN, C408.1, C409.1, C410.1, C411.1, C412.1, C413.1, C414.1, C415.1, C416.1, C417.1, C418.1, C419.1, C420.1, J400.2, R400.2, RV400.E, SJ400.1, SJ401.1, SW408.2, U400.AVDD, U400.VDD, U401.3V3OUT, U401.VCC, U401.VCCIO, U402.V+, U404M.VCC, XDS400.VDD
- net 5V: now also J402A.P$1, J403B.P$1, J404B.P$1, SJ401.3, SJ404.3
- net AMP_!CLIP: now also U400.RF8
- net AMP_!FAULT: now also U400.RA3
- net AMP_!OTW: now also U400.RA2
- net AMP_!RESET: now also U400.RA4
- net DSP_!BKND_ERR: now also U400.RF5
- net DSP_!MUTE: now also U400.RD9
- net DSP_!PDN: now also U400.RD10
- net DSP_!RESET: now also U400.RD11
- net DSP_EMO1: now also U400.RD0
- net DSP_SCL: now also U400.RA14
- net DSP_SDA: now also U400.RA15
- net DSP_VALID: now also U400.RF4
- net GND: now also A400.GND, C400.2, C401.1, C402.1, C403.1, C404.1, C405.1, C406.1, C407.1, C408.2, C409.2, C410.2, C411.2, C412.2, C413.2, C414.2, C415.2, C416.2, C417.2, C418.2, C419.2, C420.2, C421.1, C422.1, J400.3, J403A.P$1, J404A.P$1, J405.GND, J406.GND, J407.GND, Q400.S, Q401.S, Q402.S, Q403.S, Q404.S, Q405.S, Q406.S, R402.1, R403.1, R405.1, RV400.A, SJ400.3, SJ403.1, SW400.2, SW401.2, SW402.2, SW403.2, SW404.2, SW405.2, SW406.2, SW407.P, U400.AVSS, U400.VSS, U401.GND, U401.GND@1, U402.V-, U404M.!OE, U404M.GND, XDS400.GND
- net I2S_LRCLK: now also A400.RFS1, U400.RD12
- net I2S_SCLK: now also A400.SCLK1, U400.RD1
- net I2S_SD: now also A400.DT1, U400.RD2
- net VBAT: now also R404.2
Other:
- moved on the sheet: A400

Commit message: Testpads added, schematic done (barring oversights)
Parts:
- added D400: D5V0L2B3SO, BW-Active:SOT23-TVS
- added D401, D402, D403, D404: BAT60A, BW-Active:SOD323-SCHOTTKY
- added J408: AUX, BW-Connectors:GEN-4PIN
- added R407, R408, R409, R410: 10kΩ, resistor:R-US_R0603
- added RV401: 10kΩ, BW-PassiveMechanical:TC33X-2
- added SW409: RESET, BW-PassiveMechanical:WIRED-SWITCH-NO
- added T312, TP100, TP101, TP102, TP103, TP104, TP105, TP106, TP200, TP201, TP202, TP203, TP204, TP300, TP301, TP302, TP303, TP304, TP305, TP306, TP307, TP308, TP309, TP310, TP311, TP313, TP314, TP315, TP316, TP317, TP318, TP319, TP320, TP321, TP322, TP323, TP324, TP325, TP326, TP400, TP401, TP402, TP403, TP404, TP405, TP406, TP407, TP408, TP409, TP410, TP411, TP412, TP413: TPTP15R, testpad:TPTP15R
- C221, C408: device rcl:C-EUC0805 -> rcl:C-EUC0603
- U402: value NCS20071 -> NCS4333; device BW-Active:NCS20071 -> BW-Active:NCS4333
Connections:
- new net BAT_CSN_BUF: R409.2, U402C.-IN, U402C.OUT
- new net BAT_CSP_BUF: R408.2, U402D.-IN, U402D.OUT
- new net BM_AUX_L: A400.AIL, D400.1, J408C.P$1
- new net BM_AUX_R: A400.AIR, D400.2, J408B.P$1
- new net LCD_V0: RV401.S, XDS400.NC1
- new net MCU_AUX_DETECT: J408D.P$1, U400.RC14
- new net MCU_CURR_SENSE: D402.A, D404.C, R407.1, TP409.TP, U400.RB7, U402B.OUT
- new net MCU_CURR_SENSE_+: R409.1, R410.2, U402B.+IN
- new net MCU_CURR_SENSE_-: R407.2, R408.1, U402B.-IN
- net 12V: now also TP201.TP
- net 3.3V: now also D401.C, D402.C, RV401.E, TP204.TP, U402A.V+; no longer U402.V+
- net 3.6V: now also TP203.TP
- net 5V: now also TP202.TP
- net AMP_!CLIP: now also TP326.TP
- net AMP_!FAULT: now also TP324.TP
- net AMP_!OTW: now also TP325.TP
- net AMP_!RESET: now also TP323.TP
- net AMP_AVDD: now also TP310.TP
- net AMP_A_FUSED: now also TP315.TP
- net AMP_B_FILT: now also TP316.TP
- net AMP_C_FUSED: now also TP317.TP
- net AMP_DVDD: now also TP309.TP
- net AMP_D_FILT: now also TP318.TP
- net AMP_FAN_+: now also TP320.TP
- net AMP_FAN_SENSE: now also TP319.TP
- net AMP_OUT_A: now also TP311.TP
- net AMP_OUT_B: now also T312.TP
- net AMP_OUT_C: now also TP313.TP
- net AMP_OUT_D: now also TP314.TP
- net AMP_PVDD: now also TP200.TP
- net BAT-: now also R405.1, R410.1, TP103.TP, U402A.V-
- net BAT_CSN: now also U402C.+IN
- net BAT_CSP: now also U402D.+IN
- net BM_!RST: now also TP413.TP
- net BM_MFB: now also TP412.TP
- net BM_UART_RXD: now also TP410.TP
- net BM_UART_TXD: now also TP411.TP
- net CHG_!FASTCHG: now also TP105.TP, U400.RB9
- net CHG_!FAULT: now also TP106.TP, U400.RB10
- net CHG_!FULLCHG: now also TP104.TP, U400.RB8
- net DSP_!BKND_ERR: now also TP322.TP
- net DSP_!MUTE: now also TP303.TP
- net DSP_!PDN: now also TP302.TP
- net DSP_!RESET: now also TP301.TP
- net DSP_EMO1: now also TP300.TP
- net DSP_SCL: now also TP305.TP
- net DSP_SDA: now also TP304.TP
- net DSP_VALID: now also TP321.TP
- net GND: now also D400.C, D403.A, D404.A, J408A.P$1, RV401.A, SW409.1; no longer R405.1, U402.V-
- net I2S_LRCLK: now also TP306.TP
- net I2S_SCLK: now also TP307.TP
- net I2S_SD: now also TP308.TP
- net LCD_!CS: now also TP404.TP
- net LCD_!INT: now also TP406.TP
- net LCD_!PD: now also TP405.TP
- net LCD_BL_CTL: now also TP407.TP
- net LCD_MISO: now also TP402.TP
- net LCD_MOSI: now also TP403.TP
- net LCD_SCK: now also TP401.TP
- net MCU_!MCLR: now also TP400.TP
- net MCU_!MCLR!_FILT: now also SW409.2
- net MCU_BAT_SENSE: now also D401.A, D403.C, TP408.TP, U402A.-IN, U402A.OUT; no longer U402.-IN, U402.OUT
- net MCU_BAT_VDIV: now also U402A.+IN; no longer U402.+IN
- net VBAT: now also TP101.TP
- net VIN_EXT_FUSED: now also TP100.TP
- net VSUP: now also TP102.TP
Other:
- moved on the sheet: C338, C339, C419, R310, R404, R405, Y300

Commit message: Some oversights fixed, minor additions.
Parts:
- added C344: 1mF 16V, rcl:CPOL-EUE5-10.5
- C200: value 1mF -> 1mF 50V
- R407, R410: value 10kΩ -> 110kΩ 0.1%
- R408, R409: value 10kΩ -> 1kΩ 0.1%
- renumbered T312 to TP312, U404 to U403
Connections:
- net 12V: now also C344.+
- net GND: now also C344.-

Commit message: Test pads named, board started
Parts:
- TP100: TP_SIGNAL_NAME (none) -> VIN
- TP101: TP_SIGNAL_NAME (none) -> VBAT
- TP102: TP_SIGNAL_NAME (none) -> VSUP
- TP103: TP_SIGNAL_NAME (none) -> BAT-
- TP104: TP_SIGNAL_NAME (none) -> !FULLCHG
- TP105: TP_SIGNAL_NAME (none) -> !FASTCHG
- TP106: TP_SIGNAL_NAME (none) -> CHG_!FAULT
- TP200: TP_SIGNAL_NAME (none) -> PVDD
- TP201: TP_SIGNAL_NAME (none) -> 12V
- TP202: TP_SIGNAL_NAME (none) -> 5V
- TP203: TP_SIGNAL_NAME (none) -> 3.6V
- TP204: TP_SIGNAL_NAME (none) -> 3.3V
- TP300: TP_SIGNAL_NAME (none) -> EMO1
- TP301: TP_SIGNAL_NAME (none) -> DSP_!RESET
- TP302: TP_SIGNAL_NAME (none) -> DSP_!PDN
- TP303: TP_SIGNAL_NAME (none) -> !MUTE
- TP304: TP_SIGNAL_NAME (none) -> SDA
- TP305: TP_SIGNAL_NAME (none) -> SCL
- TP306: TP_SIGNAL_NAME (none) -> LRCLK
- TP307: TP_SIGNAL_NAME (none) -> SCLK
- TP308: TP_SIGNAL_NAME (none) -> SD
- TP309: TP_SIGNAL_NAME (none) -> AMP_DVDD
- TP310: TP_SIGNAL_NAME (none) -> AMP_AVDD
- TP311: TP_SIGNAL_NAME (none) -> OUT_A
- TP312: TP_SIGNAL_NAME (none) -> OUT_B
- TP313: TP_SIGNAL_NAME (none) -> OUT_C
- TP314: TP_SIGNAL_NAME (none) -> OUT_D
- TP315: TP_SIGNAL_NAME (none) -> SPK_A
- TP316: TP_SIGNAL_NAME (none) -> SPK_B
- TP317: TP_SIGNAL_NAME (none) -> SPK_C
- TP318: TP_SIGNAL_NAME (none) -> SPK_D
- TP319: TP_SIGNAL_NAME (none) -> THERM
- TP320: TP_SIGNAL_NAME (none) -> FAN
- TP321: TP_SIGNAL_NAME (none) -> VALID
- TP322: TP_SIGNAL_NAME (none) -> !BKND_ERR
- TP323: TP_SIGNAL_NAME (none) -> AMP_!RESET
- TP324: TP_SIGNAL_NAME (none) -> AMP_!FAULT
- TP325: TP_SIGNAL_NAME (none) -> !OTW
- TP326: TP_SIGNAL_NAME (none) -> !CLIP
- TP400: TP_SIGNAL_NAME (none) -> !MCLR
- TP401: TP_SIGNAL_NAME (none) -> SCK
- TP402: TP_SIGNAL_NAME (none) -> MISO
- TP403: TP_SIGNAL_NAME (none) -> MOSI
- TP404: TP_SIGNAL_NAME (none) -> !CS
- TP405: TP_SIGNAL_NAME (none) -> LCD_!PD
- TP406: TP_SIGNAL_NAME (none) -> !INT
- TP407: TP_SIGNAL_NAME (none) -> BL_CTL
- TP408: TP_SIGNAL_NAME (none) -> BATT_SENSE
- TP409: TP_SIGNAL_NAME (none) -> CURR_SENSE
- TP410: TP_SIGNAL_NAME (none) -> BM_RX
- TP411: TP_SIGNAL_NAME (none) -> BM_TX
- TP412: TP_SIGNAL_NAME (none) -> MFB
- TP413: TP_SIGNAL_NAME (none) -> BM_!RST
Connections:
- net AMP_B_FILT: now also C301.1; no longer C301.2
- net AMP_D_FILT: now also C303.1; no longer C303.2
- net AMP_PVDD: now also U301.PVDD_CD
- net GND: now also C301.2, C303.2; no longer C301.1, C303.1
Other:
- moved on the sheet: C301, C303

Commit message: Major PCB progress, about to shrink PCB (safety commit)
Parts:
- removed TP325, TP326: TPTP15R, testpad:TPTP15R
- TP309: TP_SIGNAL_NAME AMP_DVDD -> !OTW
- TP310: TP_SIGNAL_NAME AMP_AVDD -> !CLIP
Connections:
- net AMP_!CLIP: now also TP310.TP; no longer TP326.TP
- net AMP_!OTW: now also TP309.TP; no longer TP325.TP
- net AMP_AVDD: no longer TP310.TP
- net AMP_DVDD: no longer TP309.TP
Other:
- moved on the sheet: TP309, TP310
Changed lines of the file:
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@@
 <attribute name="TP_SIGNAL_NAME" value="SD"/>
 </part>
-<part name="TP309" library="testpad" library_urn="urn:adsk.eagle:library:385" deviceset="TP" device="TP15R" package3d_urn="urn:adsk.eagle:package:27968/1">
-<attribute name="TP_SIGNAL_NAME" value="AMP_DVDD"/>
-</part>
-<part name="TP310" library="testpad" library_urn="urn:adsk.eagle:library:385" deviceset="TP" device="TP15R" package3d_urn="urn:adsk.eagle:package:27968/1">
-<attribute name="TP_SIGNAL_NAME" value="AMP_AVDD"/>
-</part>
 <part name="TP311" library="testpad" library_urn="urn:adsk.eagle:library:385" deviceset="TP" device="TP15R" package3d_urn="urn:adsk.eagle:package:27968/1">
 <attribute name="TP_SIGNAL_NAME" value="OUT_A"/>
@@
 <attribute name="TP_SIGNAL_NAME" value="AMP_!FAULT"/>
 </part>
-<part name="TP325" library="testpad" library_urn="urn:adsk.eagle:library:385" deviceset="TP" device="TP15R" package3d_urn="urn:adsk.eagle:package:27968/1">
+<part name="TP309" library="testpad" library_urn="urn:adsk.eagle:library:385" deviceset="TP" device="TP15R" package3d_urn="urn:adsk.eagle:package:27968/1">
 <attribute name="TP_SIGNAL_NAME" value="!OTW"/>
 </part>
-<part name="TP326" library="testpad" library_urn="urn:adsk.eagle:library:385" deviceset="TP" device="TP15R" package3d_urn="urn:adsk.eagle:package:27968/1">
+<part name="TP310" library="testpad" library_urn="urn:adsk.eagle:library:385" deviceset="TP" device="TP15R" package3d_urn="urn:adsk.eagle:package:27968/1">
 <attribute name="TP_SIGNAL_NAME" value="!CLIP"/>
 </part>
@@
 <attribute name="NAME" x="-168.91" y="36.83" size="1.778" layer="95"/>
 </instance>
-<instance part="TP309" gate="G$1" x="55.88" y="58.42" smashed="yes" rot="R270">
-<attribute name="NAME" x="57.15" y="59.69" size="1.778" layer="95" rot="R270"/>
-</instance>
-<instance part="TP310" gate="G$1" x="66.04" y="55.88" smashed="yes">
-<attribute name="NAME" x="64.77" y="57.15" size="1.778" layer="95"/>
-</instance>
 <instance part="TP311" gate="G$1" x="157.48" y="93.98" smashed="yes">
 <attribute name="NAME" x="156.21" y="95.25" size="1.778" layer="95"/>
@@
 <attribute name="NAME" x="24.13" y="49.53" size="1.778" layer="95"/>
 </instance>
-<instance part="TP325" gate="G$1" x="27.94" y="45.72" smashed="yes">
+<instance part="TP309" gate="G$1" x="27.94" y="45.72" smashed="yes">
 <attribute name="NAME" x="26.67" y="46.99" size="1.778" layer="95"/>
 </instance>
-<instance part="TP326" gate="G$1" x="30.48" y="43.18" smashed="yes">
+<instance part="TP310" gate="G$1" x="30.48" y="43.18" smashed="yes">
 <attribute name="NAME" x="29.21" y="44.45" size="1.778" layer="95"/>
 </instance>
@@
 <pinref part="U301" gate="G$1" pin="AVDD"/>
 <wire x1="60.96" y1="27.94" x2="60.96" y2="53.34" width="0.1524" layer="91"/>
-<wire x1="60.96" y1="53.34" x2="66.04" y2="53.34" width="0.1524" layer="91"/>
-<pinref part="TP310" gate="G$1" pin="TP"/>
-<wire x1="66.04" y1="53.34" x2="83.82" y2="53.34" width="0.1524" layer="91"/>
-<junction x="66.04" y="53.34"/>
+<wire x1="60.96" y1="53.34" x2="83.82" y2="53.34" width="0.1524" layer="91"/>
 </segment>
 </net>
@@
 <pinref part="C326" gate="G$1" pin="1"/>
 <pinref part="U301" gate="G$1" pin="DVDD"/>
-<wire x1="53.34" y1="27.94" x2="53.34" y2="58.42" width="0.1524" layer="91"/>
-<wire x1="53.34" y1="58.42" x2="53.34" y2="60.96" width="0.1524" layer="91"/>
+<wire x1="53.34" y1="27.94" x2="53.34" y2="60.96" width="0.1524" layer="91"/>
 <wire x1="53.34" y1="60.96" x2="53.34" y2="66.04" width="0.1524" layer="91"/>
 <wire x1="53.34" y1="66.04" x2="83.82" y2="66.04" width="0.1524" layer="91"/>
@@
 <junction x="53.34" y="60.96"/>
 <label x="55.88" y="60.96" size="1.778" layer="95"/>
-<pinref part="TP309" gate="G$1" pin="TP"/>
-<junction x="53.34" y="58.42"/>
 </segment>
 <segment>
@@
 <wire x1="83.82" y1="43.18" x2="27.94" y2="43.18" width="0.1524" layer="91"/>
 <label x="-43.18" y="43.18" size="1.778" layer="95"/>
-<pinref part="TP325" gate="G$1" pin="TP"/>
+<pinref part="TP309" gate="G$1" pin="TP"/>
 <wire x1="27.94" y1="43.18" x2="-27.94" y2="43.18" width="0.1524" layer="91"/>
 <junction x="27.94" y="43.18"/>
@@
 <wire x1="83.82" y1="40.64" x2="30.48" y2="40.64" width="0.1524" layer="91"/>
 <label x="-43.18" y="40.64" size="1.778" layer="95"/>
-<pinref part="TP326" gate="G$1" pin="TP"/>
+<pinref part="TP310" gate="G$1" pin="TP"/>
 <wire x1="30.48" y1="40.64" x2="-27.94" y2="40.64" width="0.1524" layer="91"/>
 <junction x="30.48" y="40.64"/>

Commit message: PCB initially completed, final fixes
Parts:
- removed C417, C418, C419, C420: 0.1µF, rcl:C-EUC0603
- removed C421, C422: 18pF, rcl:C-EUC0603
- removed D401, D402, D403, D404: BAT60A, BW-Active:SOD323-SCHOTTKY
- removed J407: ZX62D-B-5PA8, BW-Connectors:ZX62D-B-5PA8
- removed SJ403: FTRESET, jumper:SJ
- removed SJ404: USB-5V, jumper:SJ2W
- removed TP322, TP323, TP324, TP401, TP402, TP403, TP404, TP405, TP406, TP407: TPTP15R, testpad:TPTP15R
- added R411, R412: 10kΩ, resistor:R-US_R0603
- added R413, R414: 1kΩ, resistor:R-US_R0603
- added U404: NCS2333, BW-Active:NCS2333
- C401, C402, C403, C404, C407: value 15pF -> 0.1µF
- C405, C406: value 15pF -> 18pF
- SJ400: value USB -> USB-5V
- TP309: TP_SIGNAL_NAME !OTW -> VALID
- TP310: TP_SIGNAL_NAME !CLIP -> !BKND_ERR
- TP321: TP_SIGNAL_NAME VALID -> AMP_!RESET
- U400: value PIC32MZ-EF-100-I/PF -> PIC32MZ-EF-100
- U402: value NCS4333 -> NCS2333; device BW-Active:NCS4333 -> BW-Active:NCS2333
Connections:
- removed net BAT_CSN_BUF: R409.2, U402C.-IN, U402C.OUT
- removed net BAT_CSP_BUF: R408.2, U402D.-IN, U402D.OUT
- removed net FT_!RESET: SJ403.2, U401.!RESET
- removed net MCU_USBID: J407.ID, U400.RF3
- removed net MCU_USB_D+: J407.D+, U400.D+
- removed net MCU_USB_D-: J407.D-, U400.D-
- removed net MCU_USB_VBUS: J407.VBUS, U400.VBUS
- removed net MCU_VUSB3V3: SJ400.2, U400.VUSB3V3
- new net MCU_BAT_SENSE_BUF: C404.1, TP408.TP, U400.RB6, U404B.-IN, U404B.OUT
- new net MCU_BAT_SENSE_FB: R411.1, U402A.-IN, U402A.OUT
- new net MCU_CURR_SENSE_BUF: C403.1, TP409.TP, U400.RB7, U404A.-IN, U404A.OUT
- new net MCU_CURR_SENSE_FB: R407.1, R412.2, U402B.OUT
- net 3.3V: now also C401.1, C402.1, C407.1, R413.2, R414.2, U404A.V+; no longer C417.1, C418.1, C419.1, C420.1, D401.C, D402.C, SJ400.1
- net 5V: now also SJ400.3; no longer SJ404.3
- net AMP_!CLIP: no longer TP310.TP
- net AMP_!FAULT: no longer TP324.TP
- net AMP_!OTW: no longer TP309.TP
- net AMP_!RESET: now also TP321.TP; no longer TP323.TP
- net BAT-: now also C402.2
- net BAT_CSN: now also R409.2; no longer U402C.+IN
- net BAT_CSP: now also R408.2; no longer U402D.+IN
- net BM_ADAP_IN: now also SJ400.2; no longer SJ404.2
- net BM_USB_VBUS: now also SJ400.1; no longer SJ404.1
- net DSP_!BKND_ERR: now also TP310.TP; no longer TP322.TP
- net DSP_SCL: now also R414.1
- net DSP_SDA: now also R413.1
- net DSP_VALID: now also TP309.TP; no longer TP321.TP
- net GND: now also C401.2, C403.2, C404.2, C407.2, U400.VUSB3V3, U404A.V-; no longer C401.1, C402.1, C403.1, C404.1, C407.1, C417.2, C418.2, C419.2, C420.2, C421.1, C422.1, D403.A, D404.A, J407.GND, SJ400.3, SJ403.1
- net LCD_!CS: no longer TP404.TP
- net LCD_!INT: no longer TP406.TP
- net LCD_!PD: no longer TP405.TP
- net LCD_BL_CTL: no longer TP407.TP
- net LCD_MISO: no longer TP402.TP
- net LCD_MOSI: no longer TP403.TP
- net LCD_SCK: no longer TP401.TP
- net MCU_BACK_SW: no longer C404.2
- net MCU_BAT_SENSE: now also R411.2, U404B.+IN; no longer D401.A, D403.C, TP408.TP, U400.RB6, U402A.-IN, U402A.OUT
- net MCU_CURR_SENSE: now also R412.1, U404A.+IN; no longer D402.A, D404.C, R407.1, TP409.TP, U400.RB7, U402B.OUT
- net MCU_FWD_SW: no longer C402.2
- net MCU_LCD_BL_SW: no longer C401.2
- net MCU_MFB_SW: no longer C406.2
- net MCU_OSC1: now also C405.2; no longer C421.2
- net MCU_OSC2_R: now also C406.2; no longer C422.2
- net MCU_PLAY_SW: no longer C403.2
- net MCU_VOL+_SW: no longer C405.2
- net MCU_VOL-_SW: no longer C407.2
Other:
- moved on the sheet: C401, C402, C403, C404, C405, C406, C407, SJ400, TP309, TP310, TP321, TP408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
