File: BlockBox v2.sch (EAGLE design)
At the start: 347 parts, among them J100 TE-770966, J400 ICSP, J401 LED, J402 SWLED, J403 USB1, J404 USB2, J405 ZX62D-B-5PA8, J406 ZX62D-B-5PA8, J408 AUX, Q100 TK3R1E04PL, Q101 TK3R1E04PL, Q102 IPP052N06L3 G, Q103 IPP052N06L3 G, Q104 IPP052N06L3 G, Q105 IPP052N06L3 G, Q106 TK3R1E04PL, Q200 SUP90142E-GE3, Q201 SUP90142E-GE3, Q202 BUK9Y43-60E, Q203 DMP4065S, Q400 DMG2302UK, Q401 DMG2302UK, Q402 DMG2302UK, Q403 DMG2302UK, Q404 NMOS, Q405 NMOS, Q406 NMOS, SW100 PWRSW, SW400 VOL-, SW401 MFB, SW402 VOL+, SW403 BACK, SW404 PLAY, SW405 FWD, SW406 LCD_BL, SW407 LEDMODE, SW408 SDA01H1S, SW409 RESET, U100 BQ77915, U101 MAX1737, U102 LM74700-Q1, U103 LM74700-Q1, U104 LM74700-Q1, U200 LM5022, U201 LM3488, U202 LM25085, U203 TPS54308, U204 LD39150DT33, U300 TAS5548, U301 TAS5634, U302 NCS20071, U400 PIC32MZ-EF-100, U401 FT230XS, U402 NCS2333, U403 FSAL200MTC, U404 NCS2333, Y300 12.288MHz, Y400 12MHz

Commit message: Added logo and ground TPs
Parts:
- added TP107, TP108, TP109: TPTP15R, testpad:TPTP15R
Connections:
- net GND: now also TP107.TP, TP108.TP, TP109.TP
Changed lines of the file:
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@@
 <part name="R413" library="resistor" library_urn="urn:adsk.eagle:library:348" deviceset="R-US_" device="R0603" package3d_urn="urn:adsk.eagle:package:23555/3" value="1kΩ"/>
 <part name="R414" library="resistor" library_urn="urn:adsk.eagle:library:348" deviceset="R-US_" device="R0603" package3d_urn="urn:adsk.eagle:package:23555/3" value="1kΩ"/>
+<part name="TP107" library="testpad" library_urn="urn:adsk.eagle:library:385" deviceset="TP" device="TP15R" package3d_urn="urn:adsk.eagle:package:27968/1">
+<attribute name="TP_SIGNAL_NAME" value="BAT-"/>
+</part>
+<part name="TP108" library="testpad" library_urn="urn:adsk.eagle:library:385" deviceset="TP" device="TP15R" package3d_urn="urn:adsk.eagle:package:27968/1">
+<attribute name="TP_SIGNAL_NAME" value="BAT-"/>
+</part>
+<part name="TP109" library="testpad" library_urn="urn:adsk.eagle:library:385" deviceset="TP" device="TP15R" package3d_urn="urn:adsk.eagle:package:27968/1">
+<attribute name="TP_SIGNAL_NAME" value="BAT-"/>
+</part>
 </parts>
 <sheets>
@@
 <instance part="TP106" gate="G$1" x="5.08" y="63.5" smashed="yes">
 <attribute name="NAME" x="3.81" y="64.77" size="1.778" layer="95"/>
+</instance>
+<instance part="TP107" gate="G$1" x="223.52" y="7.62" smashed="yes">
+<attribute name="NAME" x="219.71" y="8.89" size="1.778" layer="95"/>
+</instance>
+<instance part="TP108" gate="G$1" x="231.14" y="7.62" smashed="yes">
+<attribute name="NAME" x="229.87" y="8.89" size="1.778" layer="95"/>
+</instance>
+<instance part="TP109" gate="G$1" x="241.3" y="7.62" smashed="yes">
+<attribute name="NAME" x="240.03" y="8.89" size="1.778" layer="95"/>
 </instance>
 </instances>
@@
 <pinref part="D102" gate="G$1" pin="A"/>
 <wire x1="248.92" y1="25.4" x2="248.92" y2="5.08" width="0.1524" layer="91"/>
-<wire x1="248.92" y1="5.08" x2="218.44" y2="5.08" width="0.1524" layer="91"/>
-</segment>
-<segment>
+<wire x1="248.92" y1="5.08" x2="241.3" y2="5.08" width="0.1524" layer="91"/>
+<pinref part="TP107" gate="G$1" pin="TP"/>
+<wire x1="241.3" y1="5.08" x2="231.14" y2="5.08" width="0.1524" layer="91"/>
+<wire x1="231.14" y1="5.08" x2="223.52" y2="5.08" width="0.1524" layer="91"/>
+<wire x1="223.52" y1="5.08" x2="218.44" y2="5.08" width="0.1524" layer="91"/>
+<junction x="223.52" y="5.08"/>
+<pinref part="TP108" gate="G$1" pin="TP"/>
+<junction x="231.14" y="5.08"/>
+<pinref part="TP109" gate="G$1" pin="TP"/>
+<junction x="241.3" y="5.08"/>
+</segment>
+<segment>
